File: CGA_1_6.sch (KiCad schematic (older format))
At the start: 19 parts, among them U13 74LS08, U14 74S32, U28 74LS10, U38 MC6845, U48 74LS51, U49 74LS02, U50 2118, U51 2118, U52 2118, U53 2118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

Commit message: U28 is 74S10 and not 74LS10 in original board
Parts:
- U28: value 74LS10 -> 74S10
Changed lines of the file:
@@
 P 2800 2100
 F 0 "U28" H 2800 2425 50  0000 C CNN
-F 1 "74LS10" H 2800 2334 50  0000 C CNN
+F 1 "74S10" H 2800 2334 50  0000 C CNN
 F 2 "Package_DIP:DIP-14_W7.62mm_LongPads" H 2800 2100 50  0001 C CNN
 F 3 "http://www.ti.com/lit/gpn/sn74LS10" H 2800 2100 50  0001 C CNN
