File: CGA_4_6.sch (KiCad schematic (older format))
At the start: 20 parts, among them U1 74S112, U15 74LS00, U16 74LS04, U2 74LS74, U20 74LS04, U22 74LS51, U23 74LS32, U25 74LS00, U26 74S04, U27 74LS51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

Commit message: U28 is 74S10 and not 74LS10 in original board
Parts:
- U28: value 74LS10 -> 74S10
Changed lines of the file:
@@
 P 5500 3900
 F 0 "U28" H 5500 3583 50  0000 C CNN
-F 1 "74LS10" H 5500 3674 50  0000 C CNN
+F 1 "74S10" H 5500 3674 50  0000 C CNN
 F 2 "Package_DIP:DIP-14_W7.62mm_LongPads" H 5500 3900 50  0001 C CNN
 F 3 "http://www.ti.com/lit/gpn/sn74LS10" H 5500 3900 50  0001 C CNN
@@
 AR Path="/60463CC5/63279063" Ref="U28"  Part="1"
 F 0 "U28" H 9050 7025 50  0000 C CNN
-F 1 "74LS10" H 9050 6934 50  0000 C CNN
+F 1 "74S10" H 9050 6934 50  0000 C CNN
 F 2 "Package_DIP:DIP-14_W7.62mm_LongPads" H 9050 6700 50  0001 C CNN
 F 3 "http://www.ti.com/lit/gpn/sn74LS10" H 9050 6700 50  0001 C CNN
